Commit message: ENH: fix urdf

File: src/rf_robot/urdf/fishbot_gazebo.urdf (robot description, URDF)
Before this commit: robot fishbot, 7 links, 6 joints
Links:
- added link caster_link1, mass 0.02; collision sphere radius=0.016; visual sphere radius=0.016
Joints:
- added joint caster_joint1: type fixed, parent base_link, child caster_link1, origin xyz=-0.07 0.0 -0.076, axis 0 1 0
- joint caster_joint: origin xyz=0.06 0.0 -0.076 -> xyz=0.07 0.0 -0.076
